Commit message: fix real slam

File: n_turtle_ws/src/n_turtle_description/urdf/n_turtle.urdf (robot description, URDF)
Before this commit: robot turtlebot3_burger, 8 links, 7 joints
Links:
- removed link base_scan
- added link laser, mass 0.114; collision cylinder length=0.0315 radius=0.055; visual mesh filename=package://turtlebot3_description/meshes/sensors/lds.stl scale=0.001 0.001 0.001
Joints:
- joint scan_joint: child base_scan -> laser
